Commit message: Added a xacro file to understand the difference between URDF & XACRO

File: unitree_a1_description/urdf/unitreeA1.urdf (robot description, URDF)
Before this commit: robot unitreeA1, 15 links, 14 joints
Joints:
- joint back_left_hip_to_trunk: axis 1 0 0 -> 1 0 1
- joint back_right_hip_to_trunk: axis 1 0 0.0 -> 1 0 1
- joint front_left_hip_to_trunk: axis 1 0 0.0 -> 1 0 1
- joint front_right_hip_to_trunk: axis 1 0 0 -> 1 0 1
